File: KiCad/K6802-SBC.kicad_sch (KiCad schematic)
At the start: 47 parts, among them J1 Barrel_Jack_Switch, J2 SBC6303 BUS, J3 SERIAL JP, SW1 POWER, SW2 RESET, U1 74LS00, U2 74LS00, U3 MC6802, U4 74LS138, U5 HM628128D_DIP32_SOP32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

Commit message: プリントパターン作成、ガーバーデータ出力
Parts:
- C1, C10, C11, C12, C13, C14, C2, C4, C6, C7, C8, C9: footprint (none) -> Capacitor_THT:C_Disc_D3.0mm_W2.0mm_P2.50mm
- C3, C5: footprint (none) -> Capacitor_THT:CP_Radial_D5.0mm_P2.50mm
- D1: footprint (none) -> Diode_THT:D_A-405_P10.16mm_Horizontal
- D2: footprint (none) -> LED_THT:LED_D3.0mm
- J1: footprint (none) -> Connector_BarrelJack:BarrelJack_Horizontal
- J3: footprint (none) -> Connector_PinHeader_2.54mm:PinHeader_1x06_P2.54mm_Horizontal
- JP1, JP2, JP3, JP4, JP5: footprint (none) -> Jumper:SolderJumper-2_P1.3mm_Open_RoundedPad1.0x1.5mm
- JP6: footprint (none) -> Jumper:SolderJumper-2_P1.3mm_Bridged_RoundedPad1.0x1.5mm
- JP7, SW1: footprint (none) -> Connector_PinHeader_2.54mm:PinHeader_1x03_P2.54mm_Vertical
- R1, R3, R4: footprint (none) -> Resistor_THT:R_Axial_DIN0207_L6.3mm_D2.5mm_P10.16mm_Horizontal
- SW2: footprint (none) -> Button_Switch_THT:SW_PUSH_6mm
- U1, U2: footprint (none) -> Package_DIP:DIP-14_W7.62mm_Socket
- U3: footprint Package_DIP:DIP-40_W15.24mm -> Package_DIP:DIP-40_W15.24mm_Socket
- U4, U6: footprint (none) -> Package_DIP:DIP-16_W7.62mm_Socket
- U5: footprint (none) -> Package_DIP:DIP-32_W15.24mm_Socket
- U7: footprint Package_DIP:DIP-28_W15.24mm -> Package_DIP:DIP-28_W15.24mm_Socket
- U8: footprint Package_DIP:DIP-24_W15.24mm -> Package_DIP:DIP-24_W15.24mm_Socket
- Y1, Y2: footprint (none) -> Crystal:Crystal_HC49-U_Vertical
Connections:
- net A14: now also JP7.1 (A); no longer JP7.2 (C)
- net at U7.27 (A14): now also JP7.2 (C); no longer JP7.1 (A)
Other:
- moved on the sheet: JP7

Commit message: シリアルクロック間違い修正(回路図だけ)
Connections:
- net at R4.1: now also C9.2, U6.10 (Φ0), Y2.1; no longer U6.11 (~{Φ1})
- net at C10.2, R4.2, Y2.2: now also U6.11 (~{Φ1})
Other:
- moved on the sheet: R4
Changed lines of the file:
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@@
 	)
 	(junction
+		(at 224.79 219.71)
+		(diameter 0)
+		(color 0 0 0 0)
+	)
+	(junction
 		(at 157.48 163.83)
 		(diameter 0)
@@
 	)
 	(junction
+		(at 236.22 219.71)
+		(diameter 0)
+		(color 0 0 0 0)
+	)
+	(junction
 		(at 113.03 76.2)
 		(diameter 0)
@@
 	(wire
 		(pts
+			(xy 233.68 219.71) (xy 236.22 219.71)
+		)
+		(stroke
+			(width 0)
+			(type default)
+		)
+	)
+	(wire
+		(pts
 			(xy 69.85 245.11) (xy 71.12 245.11)
 		)
@@
 	(wire
 		(pts
-			(xy 236.22 228.6) (xy 236.22 229.87)
+			(xy 236.22 219.71) (xy 236.22 229.87)
 		)
 		(stroke
@@
 	(wire
 		(pts
+			(xy 224.79 219.71) (xy 228.6 219.71)
+		)
+		(stroke
+			(width 0)
+			(type default)
+		)
+	)
+	(wire
+		(pts
 			(xy 60.96 114.3) (xy 97.79 114.3)
 		)
@@
 	(wire
 		(pts
-			(xy 236.22 223.52) (xy 236.22 219.71)
-		)
-		(stroke
-			(width 0)
-			(type default)
-		)
-	)
-	(wire
-		(pts
 			(xy 45.72 189.23) (xy 45.72 191.77)
 		)
@@
 	(wire
 		(pts
-			(xy 224.79 229.87) (xy 224.79 217.17)
+			(xy 224.79 229.87) (xy 224.79 219.71)
 		)
 		(stroke
@@
 	(wire
 		(pts
+			(xy 224.79 219.71) (xy 224.79 217.17)
+		)
+		(stroke
+			(width 0)
+			(type default)
+		)
+	)
+	(wire
+		(pts
 			(xy 87.63 229.87) (xy 87.63 234.95)
 		)
@@
 	(symbol
 		(lib_id "Device:R_Small_US")
-		(at 236.22 226.06 0)
+		(at 231.14 219.71 90)
 		(unit 1)
 		(exclude_from_sim no)
@@
 		(dnp no)
 		(property "Reference" "R4"
-			(at 237.236 224.79 0)
+			(at 228.854 218.44 90)
 			(effects
 				(font
@@
 		)
 		(property "Value" "1M"
-			(at 236.982 227.584 0)
+			(at 234.696 221.996 90)
 			(effects
 				(font
@@
 		)
 		(property "Footprint" "Resistor_THT:R_Axial_DIN0207_L6.3mm_D2.5mm_P10.16mm_Horizontal"
-			(at 236.22 226.06 0)
+			(at 231.14 219.71 0)
 			(effects
 				(font
@@
 		)
 		(property "Datasheet" "~"
-			(at 236.22 226.06 0)
+			(at 231.14 219.71 0)
 			(effects
 				(font
@@
 		)
 		(property "Description" "Resistor, small US symbol"
-			(at 236.22 226.06 0)
+			(at 231.14 219.71 0)
 			(effects
 				(font

Commit message: $C000無効かジャンパ追加 REV2ガーバー出力
Parts:
- added JP8: C000_JP, Jumper:SolderJumper-2_P1.3mm_Open_RoundedPad1.0x1.5mm, symbol Jumper:SolderJumper_2_Open
- JP1: value C000_JP -> 16k_JP
Connections:
- net $8000: now also U2.10; no longer U2.9
- net $C000: now also JP8.1 (A)
- net GND: no longer U1.12, U1.13, U2.12, U2.13
- net at JP2.2 (B), RN1.3 (R2): now also U1.12; no longer U2.10
- net at RN1.4 (R3): now also U1.13, JP8.2 (B)
- net at U2.11: now also U2.9
- net at U1.11: now also U2.12, U2.13
- net ~{RAM_DIABLE} renamed RAM_DIABLE
- no-connect marks 20 -> 17
Other:
- moved on the sheet: JP2, U1D, U2C, U2D
